Commit message: Canadarm moveit setup (#2)
* collision meshes

Signed-off-by: Dharini Dutia <dharini@openrobotics.org>

* best path

Signed-off-by: Dharini Dutia <dharini@openrobotics.org>

* updating stls

Signed-off-by: Dharini Dutia <dharini@openrobotics.org>

---------

Signed-off-by: Dharini Dutia <dharini@openrobotics.org>

File: models/canadarm/urdf/SSRMS_Canadarm2.urdf (robot description, URDF)
Before this commit: robot SSRMS_Canadarm2, 9 links, 8 joints
Links:
- link B1: geometry collision mesh filename=file:///home/spaceros-user/demos_ws/src/simulation/models/c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 scale=1.0 1.0 1.0; visual mesh filename=file:///home/spaceros-user/demos_ws/src/simulation/models/c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 scale=1.0 1.0 1.0
- link B2: geometry collision mesh filename=file:///home/spaceros-user/demos_ws/src/simulation/models/c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 scale=1.0 1.0 1.0; visual mesh filename=file:///home/spaceros-user/demos_ws/src/simulation/models/c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 scale=1.0 1.0 1.0
- link B3: geometry collision mesh filename=file:///home/spaceros-user/demos_ws/src/simulation/models/c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 scale=1.0 1.0 1.0; collision mesh filename=file:///home/spaceros-user/demos_ws/src/simulation/models/c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 scale=1.0 1.0 1.0
- link B4: geometry collision mesh filename=file:///home/spaceros-user/demos_ws/src/simulation/models/c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 scale=1.0 1.0 1.0; collision mesh filename=file:///home/spaceros-user/demos_ws/src/simulation/models/c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 scale=1.0 1.0 1.0
- link B5: geometry collision mesh filename=file:///home/spaceros-user/demos_ws/src/simulation/models/c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 scale=1.0 1.0 1.0; visual mesh filename=file:///home/spaceros-user/demos_ws/src/simulation/models/c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 scale=1.0 1.0 1.0
- link B6: geometry collision mesh filename=file:///home/spaceros-user/demos_ws/src/simulation/models/c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 scale=1.0 1.0 1.0; visual mesh filename=file:///home/spaceros-user/demos_ws/src/simulation/models/c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 scale=1.0 1.0 1.0
- link Base_SSRMS: geometry collision mesh filename=file:///home/spaceros-user/demos_ws/src/simulation/models/c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 scale=1.0 1.0 1.0; visual mesh filename=file:///home/spaceros-user/demos_ws/src/simulation/models/c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 scale=1.0 1.0 1.0
- link EE_SSRMS: geometry collision mesh filename=file:///home/spaceros-user/demos_ws/src/simulation/models/c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 scale=1.0 1.0 1.0; visual mesh filename=file:///home/spaceros-user/demos_ws/src/simulation/models/c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 scale=1.0 1.0 1.0
