Commit message: Set interface as an argument

File: models/canadarm/urdf/SSRMS_Canadarm2.gazebo.xacro (robot description, xacro)
@@ -1,5 +1,5 @@
 <?xml version="1.0" ?>
 <robot xmlns:xacro="http://wiki.ros.org/xacro">
-  <xacro:macro name="ssrms_canadarm2_gazebo" params="">
+  <xacro:macro name="ssrms_canadarm2_gazebo" params="command_interface:=effort">
   <ros2_control name="IgnitionSystem" type="system">
       <hardware>
@@ -7,5 +7,5 @@
       </hardware>
       <joint name="Base_Joint">
-          <command_interface name="effort"/>
+          <command_interface name="${command_interface}"/>
           <state_interface name="position"/>
           <state_interface name="velocity"/>
@@ -13,5 +13,5 @@
       </joint>
       <joint name="Shoulder_Roll">
-          <command_interface name="effort"/>
+          <command_interface name="${command_interface}"/>
           <state_interface name="position"/>
           <state_interface name="velocity"/>
@@ -19,5 +19,5 @@
       </joint>
       <joint name="Shoulder_Yaw">
-          <command_interface name="effort"/>
+          <command_interface name="${command_interface}"/>
           <state_interface name="position"/>
           <state_interface name="velocity"/>
@@ -25,5 +25,5 @@
       </joint>
       <joint name="Elbow_Pitch">
-          <command_interface name="effort"/>
+          <command_interface name="${command_interface}"/>
           <state_interface name="position"/>
           <state_interface name="velocity"/>
@@ -31,5 +31,5 @@
       </joint>
       <joint name="Wrist_Pitch">
-          <command_interface name="effort"/>
+          <command_interface name="${command_interface}"/>
           <state_interface name="position"/>
           <state_interface name="velocity"/>
@@ -37,5 +37,5 @@
       </joint>
       <joint name="Wrist_Yaw">
-          <command_interface name="effort"/>
+          <command_interface name="${command_interface}"/>
           <state_interface name="position"/>
           <state_interface name="velocity"/>
@@ -43,5 +43,5 @@
       </joint>
       <joint name="Wrist_Roll">
-          <command_interface name="effort"/>
+          <command_interface name="${command_interface}"/>
           <state_interface name="position"/>
           <state_interface name="velocity"/>

File: models/canadarm/urdf/SSRMS_Canadarm2.urdf.xacro (robot description, xacro)
@@ -5,9 +5,9 @@
  -->
 <robot name="SSRMS_Canadarm2" xmlns:xacro="http://wiki.ros.org/xacro">
-  <xacro:arg name="xyz" default="0.0 0.0 2.0" />
-  <xacro:arg name="rpy" default="0.0 0.0 0.0" />
+  <xacro:arg name="xyz" default="0.5 0.0 1.5" />
+  <xacro:arg name="rpy" default="3.1416 0.0 0.0" />
   <!-- Gazebo - ROS2 Control macro -->
   <xacro:include filename="$(find simulation)/models/canadarm/urdf/SSRMS_Canadarm2.gazebo.xacro" />
-  <xacro:ssrms_canadarm2_gazebo/>
+  <xacro:ssrms_canadarm2_gazebo command_interface="position" />
   <link name="world" />
   <joint name="world_joint" type="fixed">
