Commit message: Added suggested changes: Delete commented out lines in urdf

File: models/canadarm/urdf/SSRMS_Canadarm2.urdf.xacro (robot description, xacro)
@@ -63,5 +63,4 @@
       <origin rpy="0 -1.5708 0" xyz="0.25082 0 -0.175"/>
       <geometry>
-        <!--<mesh filename="$(find simulation)/models/canadarm/meshes/joint_combine_link3.stl" scale="1.0 1.0 1.0" />-->
         <mesh filename="$(find simulation)/models/canadarm/meshes/joint_v3_0.stl" scale="1.0 1.0 1.0" />
       </geometry>
@@ -92,5 +91,4 @@
       <origin rpy="0 0 0" xyz="0.175 0 -0.25082"/>
       <geometry>
-        <!--<mesh filename="$(find simulation)/models/canadarm/meshes/joint_combine_link3.stl" scale="1.0 1.0 1.0" />-->
         <mesh filename="$(find simulation)/models/canadarm/meshes/joint_v3_0.stl" scale="1.0 1.0 1.0" />
       </geometry>
@@ -121,5 +119,4 @@
       <origin rpy="0 -1.5708 0" xyz="0.25082 0 -0.175"/>
       <geometry>
-        <!--<mesh filename="$(find simulation)/models/canadarm/meshes/joint_combine_link3.stl" scale="1.0 1.0 1.0" />-->
         <mesh filename="$(find simulation)/models/canadarm/meshes/joint_v3_0.stl" scale="1.0 1.0 1.0" />
       </geometry>
@@ -134,5 +131,4 @@
       <origin rpy="-1.5708 0 -1.5708" xyz="0.25082 0 -0.175"/>
       <geometry>
-        <!--<mesh filename="$(find simulation)/models/canadarm/meshes/long_link_v2_1_curr.stl" scale="1.0 1.0 1.0" />-->
         <mesh filename="$(find simulation)/models/canadarm/meshes/long_link_1_v3_0.stl" scale="1.0 1.0 1.0" />
       </geometry>
@@ -147,5 +143,4 @@
       <origin rpy="0 1.5708 0" xyz="7.36082 0 -0.175"/>
       <geometry>
-        <!--<mesh filename="$(find simulation)/models/canadarm/meshes/joint_combine_link3.stl" scale="1.0 1.0 1.0" />-->
         <mesh filename="$(find simulation)/models/canadarm/meshes/joint_v3_0.stl" scale="1.0 1.0 1.0" />
       </geometry>
@@ -195,5 +190,4 @@
       <origin rpy="1.57 -3.14 1.57" xyz="-7.36082 0 -0.175"/>
       <geometry>
-        <!--<mesh filename="$(find simulation)/models/canadarm/meshes/long_link_2.stl" scale="1.0 1.0 1.0" />-->
         <mesh filename="$(find simulation)/models/canadarm/meshes/long_link_2_v3_0.stl" scale="1.0 1.0 1.0" />
       </geometry>
@@ -208,5 +202,4 @@
       <origin rpy="0 -1.57 0" xyz="-7.36082 0 -0.175"/>
       <geometry>
-        <!--<mesh filename="$(find simulation)/models/canadarm/meshes/joint_combine_link3.stl" scale="1.0 1.0 1.0" />-->
         <mesh filename="$(find simulation)/models/canadarm/meshes/joint_v3_0.stl" scale="1.0 1.0 1.0" />
       </geometry>
@@ -237,5 +230,4 @@
       <origin rpy="0 -3.14 0" xyz="0 0 0"/>
       <geometry>
-        <!--<mesh filename="$(find simulation)/models/canadarm/meshes/joint_combine_link3.stl" scale="1.0 1.0 1.0" />-->
         <mesh filename="$(find simulation)/models/canadarm/meshes/joint_v3_0.stl" scale="1.0 1.0 1.0" />
       </geometry>
@@ -266,5 +258,4 @@
       <origin rpy="0 -1.5708 0" xyz="0 0 0"/>
       <geometry>
-        <!--<mesh filename="$(find simulation)/models/canadarm/meshes/joint_combine_link3.stl" scale="1.0 1.0 1.0" />-->
         <mesh filename="$(find simulation)/models/canadarm/meshes/joint_v3_0.stl" scale="1.0 1.0 1.0" />
       </geometry>

Commit message: Deleted another commented out line that was missed in the last commit

File: models/canadarm/urdf/SSRMS_Canadarm2.urdf.xacro (robot description, xacro)
@@ -177,5 +177,4 @@
       <origin rpy="0 1.5708 0" xyz="-0.25082 0 -0.175"/>
       <geometry>
-        <!--<mesh filename="$(find simulation)/models/canadarm/meshes/link_joint.stl" scale="1.0 1.0 1.0" />-->
         <mesh filename="$(find simulation)/models/canadarm/meshes/link_joint_v2_1.stl" scale="1.0 1.0 1.0" />
       </geometry>

Commit message: Changed find pkg to package://pkg so meshes are displayed in Rviz2

File: models/canadarm/urdf/SSRMS_Canadarm2.urdf.xacro (robot description, xacro)
@@ -27,5 +27,5 @@
       <origin rpy="0 0 0" xyz="0 0 0"/>
       <geometry>
-        <mesh filename="$(find simulation)/models/canadarm/meshes/ee.dae" scale="1.0 1.0 1.0" />
+        <mesh filename="package://simulation/models/canadarm/meshes/ee.dae" scale="1.0 1.0 1.0" />
       </geometry>
     </visual>
@@ -33,5 +33,5 @@
       <origin rpy="0 0 0" xyz="0 0 0"/>
       <geometry>
-        <mesh filename="$(find simulation)/models/canadarm/meshes/ee.stl" scale="1.0 1.0 1.0" />
+        <mesh filename="package://simulation/models/canadarm/meshes/ee.stl" scale="1.0 1.0 1.0" />
       </geometry>
     </collision>
@@ -57,11 +57,11 @@
       <origin rpy="0 -1.5708 0" xyz="0.25082 0 -0.175"/>
       <geometry>
-        <mesh filename="$(find simulation)/models/canadarm/meshes/joint_v3_0.dae" scale="1.0 1.0 1.0" />
-      </geometry>
-    </visual>
-    <collision>
-      <origin rpy="0 -1.5708 0" xyz="0.25082 0 -0.175"/>
-      <geometry>
-        <mesh filename="$(find simulation)/models/canadarm/meshes/joint_v3_0.stl" scale="1.0 1.0 1.0" />
+        <mesh filename="package://simulation/models/canadarm/meshes/joint_v3_0.dae" scale="1.0 1.0 1.0" />
+      </geometry>
+    </visual>
+    <collision>
+      <origin rpy="0 -1.5708 0" xyz="0.25082 0 -0.175"/>
+      <geometry>
+        <mesh filename="package://simulation/models/canadarm/meshes/joint_v3_0.stl" scale="1.0 1.0 1.0" />
       </geometry>
     </collision>
@@ -85,5 +85,5 @@
       <origin rpy="0 0 0" xyz="0.175 0 -0.25082"/>
       <geometry>
-        <mesh filename="$(find simulation)/models/canadarm/meshes/joint_v3_0.dae" scale="1.0 1.0 1.0" />
+        <mesh filename="package://simulation/models/canadarm/meshes/joint_v3_0.dae" scale="1.0 1.0 1.0" />
       </geometry>
     </visual>
@@ -91,5 +91,5 @@
       <origin rpy="0 0 0" xyz="0.175 0 -0.25082"/>
       <geometry>
-        <mesh filename="$(find simulation)/models/canadarm/meshes/joint_v3_0.stl" scale="1.0 1.0 1.0" />
+        <mesh filename="package://simulation/models/canadarm/meshes/joint_v3_0.stl" scale="1.0 1.0 1.0" />
       </geometry>
     </collision>
@@ -113,11 +113,11 @@
       <origin rpy="0 -1.5708 0" xyz="0.25082 0 -0.175"/>
       <geometry>
-        <mesh filename="$(find simulation)/models/canadarm/meshes/joint_v3_0.dae" scale="1.0 1.0 1.0" />
-      </geometry>
-    </visual>
-    <collision>
-      <origin rpy="0 -1.5708 0" xyz="0.25082 0 -0.175"/>
-      <geometry>
-        <mesh filename="$(find simulation)/models/canadarm/meshes/joint_v3_0.stl" scale="1.0 1.0 1.0" />
+        <mesh filename="package://simulation/models/canadarm/meshes/joint_v3_0.dae" scale="1.0 1.0 1.0" />
+      </geometry>
+    </visual>
+    <collision>
+      <origin rpy="0 -1.5708 0" xyz="0.25082 0 -0.175"/>
+      <geometry>
+        <mesh filename="package://simulation/models/canadarm/meshes/joint_v3_0.stl" scale="1.0 1.0 1.0" />
       </geometry>
     </collision>
@@ -125,5 +125,5 @@
       <origin rpy="-1.5708 0 -1.5708" xyz="0.25082 0 -0.175"/>
       <geometry>
-        <mesh filename="$(find simulation)/models/canadarm/meshes/long_link_1_v3_0.dae" scale="1.0 1.0 1.0" />
+        <mesh filename="package://simulation/models/canadarm/meshes/long_link_1_v3_0.dae" scale="1.0 1.0 1.0" />
       </geometry>
     </visual>
@@ -131,5 +131,5 @@
       <origin rpy="-1.5708 0 -1.5708" xyz="0.25082 0 -0.175"/>
       <geometry>
-        <mesh filename="$(find simulation)/models/canadarm/meshes/long_link_1_v3_0.stl" scale="1.0 1.0 1.0" />
+        <mesh filename="package://simulation/models/canadarm/meshes/long_link_1_v3_0.stl" scale="1.0 1.0 1.0" />
       </geometry>
     </collision>
@@ -137,5 +137,5 @@
       <origin rpy="0 1.5708 0" xyz="7.36082 0 -0.175"/>
       <geometry>
-        <mesh filename="$(find simulation)/models/canadarm/meshes/joint_v3_0.dae" scale="1.0 1.0 1.0" />
+        <mesh filename="package://simulation/models/canadarm/meshes/joint_v3_0.dae" scale="1.0 1.0 1.0" />
       </geometry>
     </visual>
@@ -143,5 +143,5 @@
       <origin rpy="0 1.5708 0" xyz="7.36082 0 -0.175"/>
       <geometry>
-        <mesh filename="$(find simulation)/models/canadarm/meshes/joint_v3_0.stl" scale="1.0 1.0 1.0" />
+        <mesh filename="package://simulation/models/canadarm/meshes/joint_v3_0.stl" scale="1.0 1.0 1.0" />
       </geometry>
     </collision>
@@ -171,5 +171,5 @@
       <origin rpy="0 1.5708 0" xyz="-0.25082 0 -0.175"/>
       <geometry>
-        <mesh filename="$(find simulation)/models/canadarm/meshes/link_joint_v2_1.dae" scale="1.0 1.0 1.0" />
+        <mesh filename="package://simulation/models/canadarm/meshes/link_joint_v2_1.dae" scale="1.0 1.0 1.0" />
       </geometry>
     </visual>
@@ -177,5 +177,5 @@
       <origin rpy="0 1.5708 0" xyz="-0.25082 0 -0.175"/>
       <geometry>
-        <mesh filename="$(find simulation)/models/canadarm/meshes/link_joint_v2_1.stl" scale="1.0 1.0 1.0" />
+        <mesh filename="package://simulation/models/canadarm/meshes/link_joint_v2_1.stl" scale="1.0 1.0 1.0" />
       </geometry>
     </collision>
@@ -183,5 +183,5 @@
       <origin rpy="1.57 -3.14 1.57" xyz="-7.36082 0 -0.175"/>
       <geometry>
-        <mesh filename="$(find simulation)/models/canadarm/meshes/long_link_2_v3_0.dae" scale="1.0 1.0 1.0" />
+        <mesh filename="package://simulation/models/canadarm/meshes/long_link_2_v3_0.dae" scale="1.0 1.0 1.0" />
       </geometry>
     </visual>
@@ -189,5 +189,5 @@
       <origin rpy="1.57 -3.14 1.57" xyz="-7.36082 0 -0.175"/>
       <geometry>
-        <mesh filename="$(find simulation)/models/canadarm/meshes/long_link_2_v3_0.stl" scale="1.0 1.0 1.0" />
+        <mesh filename="package://simulation/models/canadarm/meshes/long_link_2_v3_0.stl" scale="1.0 1.0 1.0" />
       </geometry>
     </collision>
@@ -195,5 +195,5 @@
       <origin rpy="0 -1.57 0" xyz="-7.36082 0 -0.175"/>
       <geometry>
-        <mesh filename="$(find simulation)/models/canadarm/meshes/joint_v3_0.dae" scale="1.0 1.0 1.0" />
+        <mesh filename="package://simulation/models/canadarm/meshes/joint_v3_0.dae" scale="1.0 1.0 1.0" />
       </geometry>
     </visual>
@@ -201,5 +201,5 @@
       <origin rpy="0 -1.57 0" xyz="-7.36082 0 -0.175"/>
       <geometry>
-        <mesh filename="$(find simulation)/models/canadarm/meshes/joint_v3_0.stl" scale="1.0 1.0 1.0" />
+        <mesh filename="package://simulation/models/canadarm/meshes/joint_v3_0.stl" scale="1.0 1.0 1.0" />
       </geometry>
     </collision>
@@ -223,5 +223,5 @@
       <origin rpy="0 -3.14 0" xyz="0 0 0"/>
       <geometry>
-        <mesh filename="$(find simulation)/models/canadarm/meshes/joint_v3_0.dae" scale="1.0 1.0 1.0" />
+        <mesh filename="package://simulation/models/canadarm/meshes/joint_v3_0.dae" scale="1.0 1.0 1.0" />
       </geometry>
     </visual>
@@ -229,5 +229,5 @@
       <origin rpy="0 -3.14 0" xyz="0 0 0"/>
       <geometry>
-        <mesh filename="$(find simulation)/models/canadarm/meshes/joint_v3_0.stl" scale="1.0 1.0 1.0" />
+        <mesh filename="package://simulation/models/canadarm/meshes/joint_v3_0.stl" scale="1.0 1.0 1.0" />
       </geometry>
     </collision>
@@ -251,5 +251,5 @@
       <origin rpy="0 -1.5708 0" xyz="0 0 0"/>
       <geometry>
-        <mesh filename="$(find simulation)/models/canadarm/meshes/joint_v3_0.dae" scale="1.0 1.0 1.0" />
+        <mesh filename="package://simulation/models/canadarm/meshes/joint_v3_0.dae" scale="1.0 1.0 1.0" />
       </geometry>
     </visual>
@@ -257,5 +257,5 @@
       <origin rpy="0 -1.5708 0" xyz="0 0 0"/>
       <geometry>
-        <mesh filename="$(find simulation)/models/canadarm/meshes/joint_v3_0.stl" scale="1.0 1.0 1.0" />
+        <mesh filename="package://simulation/models/canadarm/meshes/joint_v3_0.stl" scale="1.0 1.0 1.0" />
       </geometry>
     </collision>
@@ -279,5 +279,5 @@
       <origin rpy="0 -3.1415 0" xyz="0 0 0"/>
       <geometry>
-        <mesh filename="$(find simulation)/models/canadarm/meshes/ee.dae" scale="1.0 1.0 1.0" />
+        <mesh filename="package://simulation/models/canadarm/meshes/ee.dae" scale="1.0 1.0 1.0" />
       </geometry>
     </visual>
@@ -285,5 +285,5 @@
       <origin rpy="0 -3.1415 0" xyz="0 0 0"/>
       <geometry>
-        <mesh filename="$(find simulation)/models/canadarm/meshes/ee.stl" scale="1.0 1.0 1.0" />
+        <mesh filename="package://simulation/models/canadarm/meshes/ee.stl" scale="1.0 1.0 1.0" />
       </geometry>
     </collision>
