Commit message: Add base_link to mars_rover model (#11).

File: models/curiosity_path/urdf/chassis.xacro (robot description, xacro)
@@ -4,7 +4,13 @@
     <!-- Used for fixing robot to Gazebo 'chassis' -->
 	<link name="base_footprint" />
-	<joint name="base_joint" type="fixed">
+	<link name="base_link" />
+	<joint name="base_footprint_to_link" type="fixed">
 		<parent link="base_footprint"/>
+		<child link="base_link"/>
+	</joint>
+	<joint name="base_to_chassis" type="fixed">
+		<parent link="base_link"/>
 		<child link="chassis"/>
+		<origin rpy="0 0 1.57" xyz="0 0 0"/>
 	</joint>
 	<link name='chassis'>
