Commit message: Add nav camera to model and update dyn values

File: models/lunar_pole_exploration_rover/urdf/lunar_pole_exploration_rover_properties.xacro (robot description, xacro)
@@ -31,5 +31,5 @@
 	<xacro:property name="suspension_damping" value="1000.0"/>
 	<xacro:property name="suspension_friction" value="1000.0"/>
-	<xacro:property name="suspension_stiffness" value="20000.0"/>
+	<xacro:property name="suspension_stiffness" value="200000.0"/>
 	<xacro:property name="axleHeight" value="0.182"/>
 	<xacro:property name="axleWidth" value="0.1435"/>
@@ -39,7 +39,7 @@
 	<xacro:property name="axleComY" value="0.048"/>
 	<xacro:property name="axleComZ" value="0.026"/>
-	<xacro:property name="suspension_steer_limit" value="0.6"/>
-	<xacro:property name="suspension_steer_effort" value="10000.0"/>
-	<xacro:property name="suspension_steer_velocity" value="10.0"/>
+	<xacro:property name="suspension_steer_limit" value="0.7"/>
+	<xacro:property name="suspension_steer_effort" value="100000.0"/>
+	<xacro:property name="suspension_steer_velocity" value="1000.0"/>
 	<!-- Wheels properties -->
 	<xacro:property name="wheelWidth" value="0.240"/>
@@ -57,8 +57,8 @@
 	<xacro:property name="mastCameraHeight" value="0.130"/>
 	<xacro:property name="mast_camera_pan_limit" value="3.490659"/>
-	<xacro:property name="mast_camera_pan_effort" value="500.0"/>
-	<xacro:property name="mast_camera_pan_velocity" value="0.9"/>
+	<xacro:property name="mast_camera_pan_effort" value="50000.0"/>
+	<xacro:property name="mast_camera_pan_velocity" value="4.0"/>
 	<xacro:property name="mast_camera_tilt_limit" value="1.308997"/>
-	<xacro:property name="mast_camera_tilt_effort" value="500.0"/>
-	<xacro:property name="mast_camera_tilt_velocity" value="0.5"/>
+	<xacro:property name="mast_camera_tilt_effort" value="50000.0"/>
+	<xacro:property name="mast_camera_tilt_velocity" value="3.0"/>
 </robot>

File: models/lunar_pole_exploration_rover/urdf/mast_head.xacro (robot description, xacro)
@@ -88,4 +88,53 @@
             </actuator>
         </transmission>
+        <material name="green">
+            <color rgba="0 0.8 0 1"/>
+        </material>
+        <link name="nav_camera_link_left">
+            <!-- Inertial for gazebo to take it into account, Put 1gr weight -->
+            <inertial>
+                <origin xyz="0 0 0" rpy="0 0 0"/>
+                <mass value="0.001" />
+                <inertia ixx="9.1875e-09" ixy="0.0" ixz="0.0" iyy="9.1875e-09" iyz="0.0" izz="1.378125e-08"/>
+            </inertial>
+            <visual>
+                <origin rpy="0.0 0 0" xyz="0 0 0"/>
+                <geometry>
+                    <box size="0.0005 0.0005 0.0005"/>
+                </geometry>
+                <material name="green"/>
+            </visual>
+        </link>
+        <gazebo reference="nav_camera_link_left">
+            <material>Gazebo/Green</material>
+        </gazebo>
+        <joint name="nav_camera_link_left_joint" type="fixed">
+            <parent link="mast_camera"/>
+            <child link="nav_camera_link_left"/>
+            <origin xyz="0.150 0.170 0.0" rpy="0 0 0"/>
+        </joint>
+        <link name="nav_camera_link_right">
+            <!-- Inertial for gazebo to take it into account, Put 1gr weight -->
+            <inertial>
+                <origin xyz="0 0 0" rpy="0 0 0"/>
+                <mass value="0.001" />
+                <inertia ixx="9.1875e-09" ixy="0.0" ixz="0.0" iyy="9.1875e-09" iyz="0.0" izz="1.378125e-08"/>
+            </inertial>
+            <visual>
+                <origin rpy="0.0 0 0" xyz="0 0 0"/>
+                <geometry>
+                    <box size="0.0005 0.0005 0.0005"/>
+                </geometry>
+                <material name="green"/>
+            </visual>
+        </link>
+        <gazebo reference="nav_camera_link_right">
+            <material>Gazebo/Green</material>
+        </gazebo>
+        <joint name="nav_camera_link_right_joint" type="fixed">
+            <parent link="mast_camera"/>
+            <child link="nav_camera_link_right"/>
+            <origin xyz="0.150 -0.170 0.0" rpy="0 0 0"/>
+        </joint>
     </xacro:macro>
 </robot>

File: models/lunar_pole_exploration_rover/urdf/wheel_assembly.xacro (robot description, xacro)
@@ -35,5 +35,6 @@
         <parent link="chassis"/>
         <child link="${placement}_${side}_suspension"/>
-        <origin xyz="${tX*0.435} ${tY*0.255} 0.094" rpy="0 0 0"/>
+        <!-- <origin xyz="${tX*0.435} ${tY*0.255} 0.094" rpy="0 0 0"/> -->
+        <origin xyz="${tX*0.435} ${tY*0.255} 0.09" rpy="0 0 0"/>
         <limit lower="${suspension_lower_limit}" upper="${suspension_upper_limit}" effort="10000.0" velocity="100.0"/>
         <axis xyz="0 0 1"/>

Commit message: Extend steer limit

File: models/lunar_pole_exploration_rover/urdf/lunar_pole_exploration_rover_properties.xacro (robot description, xacro)
@@ -39,5 +39,5 @@
 	<xacro:property name="axleComY" value="0.048"/>
 	<xacro:property name="axleComZ" value="0.026"/>
-	<xacro:property name="suspension_steer_limit" value="0.7"/>
+	<xacro:property name="suspension_steer_limit" value="0.9"/>
 	<xacro:property name="suspension_steer_effort" value="100000.0"/>
 	<xacro:property name="suspension_steer_velocity" value="1000.0"/>
