Commit message: Fix URDF

File: models/lunar_pole_exploration_rover/urdf/chassis.xacro (robot description, xacro)
@@ -149,18 +149,30 @@
 		</inertial>
 	</link>
-	<joint name="left_solar_panel_joint" type="fixed">
+  <!-- joint is not of fixed type to avoid "lumping" from some URDF parsers
+  The joint visual need to be independant for the solar panel plugin to work -->
+  <joint name="left_solar_panel_joint" type="revolute">
     <parent link="body"/>
     <child link="left_solar_panel"/>
-    <origin xyz="0.0252 0.7253 0.3829" rpy="-1.4673 0 ${PI}"/>
+    <origin xyz="0.0252 0.7253 0.3829" rpy="1.4673 0 ${-PI}"/>
+	<axis xyz="0 0 1"/>
+    <limit lower="0.0" upper="0.0" effort="1e10" velocity="0.0"/>
   </joint>
-  <joint name="right_solar_panel_joint" type="fixed">
+  <!-- joint is not of fixed type to avoid "lumping" from some URDF parsers
+  The joint visual need to be independant for the solar panel plugin to work -->
+  <joint name="right_solar_panel_joint" type="revolute">
     <parent link="body"/>
     <child link="right_solar_panel"/>
     <origin xyz="0.0252 -0.7253 0.3829" rpy="1.4673 0 0"/>
+	<axis xyz="0 0 1"/>
+    <limit lower="0.0" upper="0.0" effort="1e10" velocity="0.0"/>
   </joint>
-  <joint name="rear_solar_panel_joint" type="fixed">
+  <!-- joint is not of fixed type to avoid "lumping" from some URDF parsers
+  The joint visual need to be independant for the solar panel plugin to work -->
+  <joint name="rear_solar_panel_joint" type="revolute">
     <parent link="body"/>
     <child link="rear_solar_panel"/>
     <origin xyz="-0.7253 0.0 0.3829" rpy="1.4673 0 ${-PI/2}"/>
+	<axis xyz="0 0 1"/>
+    <limit lower="0.0" upper="0.0" effort="1e10" velocity="0.0"/>
   </joint>
   </xacro:macro>

File: models/lunar_pole_exploration_rover/urdf/lunar_pole_exploration_rover.xacro (robot description, xacro)
@@ -16,21 +16,21 @@
 	<xacro:chassis_body/>
 	<xacro:wheel_assembly
-        placement="left"
-        side="front"
+        placement="front"
+        side="left"
         tX="1"
         tY="1"/>
 	<xacro:wheel_assembly
-        placement="left"
-        side="rear"
+        placement="rear"
+        side="left"
         tX="-1"
         tY="1"/>
 	<xacro:wheel_assembly
-        placement="right"
-        side="front"
+        placement="front"
+        side="right"
         tX="1"
         tY="-1"/>
 	<xacro:wheel_assembly
-        placement="right"
-        side="rear"
+        placement="rear"
+        side="right"
         tX="-1"
         tY="-1"/>

File: models/lunar_pole_exploration_rover/urdf/lunar_pole_exploration_rover_properties.xacro (robot description, xacro)
@@ -29,7 +29,7 @@
 	<xacro:property name="suspension_lower_limit" value="-0.0115"/>
 	<xacro:property name="suspension_upper_limit" value="0.0115"/>
-	<xacro:property name="suspension_damping" value="0.5"/>
-	<xacro:property name="suspension_friction" value="0.5"/>
-	<xacro:property name="suspension_stiffness" value="2000.0"/>
+	<xacro:property name="suspension_damping" value="1000.0"/>
+	<xacro:property name="suspension_friction" value="1000.0"/>
+	<xacro:property name="suspension_stiffness" value="20000.0"/>
 	<xacro:property name="axleHeight" value="0.182"/>
 	<xacro:property name="axleWidth" value="0.1435"/>

File: models/lunar_pole_exploration_rover/urdf/mast_head.xacro (robot description, xacro)
@@ -32,8 +32,6 @@
             <child link="mast_head_pivot"/>
             <origin xyz="0.630 0.0 1.2535" rpy="0 0 0"/>
-            <axis>
-                <xyz>0 0 1</xyz>
-                <limit lower="${-mast_camera_pan_limit}" upper="${mast_camera_pan_limit}" effort="${mast_camera_pan_effort}" velocity="${mast_camera_pan_velocity}"/>
-            </axis>
+            <axis xyz="0 0 1"/>
+            <limit lower="${-mast_camera_pan_limit}" upper="${mast_camera_pan_limit}" effort="${mast_camera_pan_effort}" velocity="${mast_camera_pan_velocity}"/>
         </joint>
         <transmission name="mast_camera_pan_trans">
@@ -77,8 +75,6 @@
             <child link="mast_camera"/>
             <origin xyz="0 0 0" rpy="0 0 0"/>
-            <axis>
-                <xyz>0 1 0</xyz>
-                <limit lower="${-mast_camera_tilt_limit}" upper="${mast_camera_tilt_limit}" effort="${mast_camera_tilt_effort}" velocity="${mast_camera_tilt_velocity}"/>
-            </axis>
+            <axis xyz="0 1 0"/>
+            <limit lower="${-mast_camera_tilt_limit}" upper="${mast_camera_tilt_limit}" effort="${mast_camera_tilt_effort}" velocity="${mast_camera_tilt_velocity}"/>
         </joint>
         <transmission name="mast_camera_tilt_trans">

File: models/lunar_pole_exploration_rover/urdf/wheel_assembly.xacro (robot description, xacro)
@@ -3,5 +3,5 @@
   <xacro:macro name="wheel_assembly" params="placement side tX tY">
     <!-- placement is either or rear -->
-    <!-- side is either ${side} side or right side -->
+    <!-- side is either left side or right side -->
     <!-- tX is either 1 for front or -1 for rear -->
     <!-- tY is either 1 for ${side} side or -1 for right side -->
@@ -35,10 +35,8 @@
         <parent link="chassis"/>
         <child link="${placement}_${side}_suspension"/>
-        <origin xyz="${tX*0.435} ${tY*0.255} 0.94" rpy="0 0 0"/>
-        <axis>
-          <xyz>0 0 1</xyz>
-          <dynamics damping="${suspension_damping}" friction="${suspension_friction}" spring_stiffness="${suspension_stiffness}"/>
-          <limit lower="${suspension_lower_limit}" upper="${suspension_upper_limit}"/>
-        </axis>
+        <origin xyz="${tX*0.435} ${tY*0.255} 0.094" rpy="0 0 0"/>
+        <limit lower="${suspension_lower_limit}" upper="${suspension_upper_limit}" effort="10000.0" velocity="100.0"/>
+        <axis xyz="0 0 1"/>
+        <dynamics damping="${suspension_damping}" friction="${suspension_friction}" spring_stiffness="${suspension_stiffness}"/>
       </joint>
       <link name='${placement}_${side}_wheel_axle'>
@@ -72,8 +70,6 @@
         <child link="${placement}_${side}_wheel_axle"/>
         <origin xyz="0.0 ${tY*0.27} -0.1265" rpy="0 0 0"/>
-        <axis>
-          <xyz>0 0 1</xyz>
-          <limit lower="${-suspension_steer_limit}" upper="${suspension_steer_limit}" effort="${suspension_steer_effort}" velocity="${suspension_steer_velocity}"/>
-        </axis>
+        <axis xyz="0 0 1"/>
+        <limit lower="${-suspension_steer_limit}" upper="${suspension_steer_limit}" effort="${suspension_steer_effort}" velocity="${suspension_steer_velocity}"/>
       </joint>
       <transmission name="${placement}_${side}_wheel_steer_trans">

Commit message: Add AftCam to rover

File: models/lunar_pole_exploration_rover/urdf/chassis.xacro (robot description, xacro)
@@ -149,31 +149,80 @@
 		</inertial>
 	</link>
-  <!-- joint is not of fixed type to avoid "lumping" from some URDF parsers
-  The joint visual need to be independant for the solar panel plugin to work -->
-  <joint name="left_solar_panel_joint" type="revolute">
-    <parent link="body"/>
-    <child link="left_solar_panel"/>
-    <origin xyz="0.0252 0.7253 0.3829" rpy="1.4673 0 ${-PI}"/>
-	<axis xyz="0 0 1"/>
-    <limit lower="0.0" upper="0.0" effort="1e10" velocity="0.0"/>
-  </joint>
-  <!-- joint is not of fixed type to avoid "lumping" from some URDF parsers
-  The joint visual need to be independant for the solar panel plugin to work -->
-  <joint name="right_solar_panel_joint" type="revolute">
-    <parent link="body"/>
-    <child link="right_solar_panel"/>
-    <origin xyz="0.0252 -0.7253 0.3829" rpy="1.4673 0 0"/>
-	<axis xyz="0 0 1"/>
-    <limit lower="0.0" upper="0.0" effort="1e10" velocity="0.0"/>
-  </joint>
-  <!-- joint is not of fixed type to avoid "lumping" from some URDF parsers
-  The joint visual need to be independant for the solar panel plugin to work -->
-  <joint name="rear_solar_panel_joint" type="revolute">
-    <parent link="body"/>
-    <child link="rear_solar_panel"/>
-    <origin xyz="-0.7253 0.0 0.3829" rpy="1.4673 0 ${-PI/2}"/>
-	<axis xyz="0 0 1"/>
-    <limit lower="0.0" upper="0.0" effort="1e10" velocity="0.0"/>
-  </joint>
+	<!-- joint is not of fixed type to avoid "lumping" from some URDF parsers
+	The joint visual need to be independant for the solar panel plugin to work -->
+	<joint name="left_solar_panel_joint" type="revolute">
+		<parent link="body"/>
+		<child link="left_solar_panel"/>
+		<origin xyz="0.0252 0.7253 0.3829" rpy="1.4673 0 ${-PI}"/>
+		<axis xyz="0 0 1"/>
+		<limit lower="0.0" upper="0.0" effort="1e10" velocity="0.0"/>
+	</joint>
+	<!-- joint is not of fixed type to avoid "lumping" from some URDF parsers
+	The joint visual need to be independant for the solar panel plugin to work -->
+	<joint name="right_solar_panel_joint" type="revolute">
+		<parent link="body"/>
+		<child link="right_solar_panel"/>
+		<origin xyz="0.0252 -0.7253 0.3829" rpy="1.4673 0 0"/>
+		<axis xyz="0 0 1"/>
+		<limit lower="0.0" upper="0.0" effort="1e10" velocity="0.0"/>
+	</joint>
+	<!-- joint is not of fixed type to avoid "lumping" from some URDF parsers
+	The joint visual need to be independant for the solar panel plugin to work -->
+	<joint name="rear_solar_panel_joint" type="revolute">
+		<parent link="body"/>
+		<child link="rear_solar_panel"/>
+		<origin xyz="-0.7253 0.0 0.3829" rpy="1.4673 0 ${-PI/2}"/>
+		<axis xyz="0 0 1"/>
+		<limit lower="0.0" upper="0.0" effort="1e10" velocity="0.0"/>
+	</joint>
+	<material name="camera_green">
+		<color rgba="0 0.8 0 1"/>
+	</material>
+	<link name="aft_camera_link_left">
+		<!-- Inertial for gazebo to take it into account, Put 1gr weight -->
+		<inertial>
+			<origin xyz="0 0 0" rpy="0 0 0"/>
+			<mass value="0.001" />
+			<inertia ixx="9.1875e-09" ixy="0.0" ixz="0.0" iyy="9.1875e-09" iyz="0.0" izz="1.378125e-08"/>
+		</inertial>
+		<visual>
+			<origin rpy="0.0 0 0" xyz="0 0 0"/>
+			<geometry>
+				<box size="0.0005 0.0005 0.0005"/>
+			</geometry>
+			<material name="camera_green"/>
+		</visual>
+	</link>
+	<gazebo reference="aft_camera_link_left">
+		<material>Gazebo/Green</material>
+	</gazebo>
+	<joint name="aft_camera_link_left_joint" type="fixed">
+		<parent link="body"/>
+		<child link="aft_camera_link_left"/>
+		<origin xyz="-0.705 -0.150 0.682" rpy="0 0 ${PI}"/>
+	</joint>
+	<link name="aft_camera_link_right">
+		<!-- Inertial for gazebo to take it into account, Put 1gr weight -->
+		<inertial>
+			<origin xyz="0 0 0" rpy="0 0 0"/>
+			<mass value="0.001" />
+			<inertia ixx="9.1875e-09" ixy="0.0" ixz="0.0" iyy="9.1875e-09" iyz="0.0" izz="1.378125e-08"/>
+		</inertial>
+		<visual>
+			<origin rpy="0.0 0 0" xyz="0 0 0"/>
+			<geometry>
+				<box size="0.0005 0.0005 0.0005"/>
+			</geometry>
+			<material name="camera_green"/>
+		</visual>
+	</link>
+	<gazebo reference="aft_camera_link_right">
+		<material>Gazebo/Green</material>
+	</gazebo>
+	<joint name="aft_camera_link_right_joint" type="fixed">
+		<parent link="body"/>
+		<child link="aft_camera_link_right"/>
+		<origin xyz="-0.705 0.150 0.682" rpy="0 0 ${PI}"/>
+	</joint>
   </xacro:macro>
 </robot>

File: models/lunar_pole_exploration_rover/urdf/mast_head.xacro (robot description, xacro)
@@ -112,5 +112,5 @@
             <parent link="mast_camera"/>
             <child link="nav_camera_link_left"/>
-            <origin xyz="0.150 0.170 0.0" rpy="0 0 0"/>
+            <origin xyz="0.150 0.190 0.0" rpy="0 0 0"/>
         </joint>
         <link name="nav_camera_link_right">
@@ -135,5 +135,5 @@
             <parent link="mast_camera"/>
             <child link="nav_camera_link_right"/>
-            <origin xyz="0.150 -0.170 0.0" rpy="0 0 0"/>
+            <origin xyz="0.150 -0.190 0.0" rpy="0 0 0"/>
         </joint>
     </xacro:macro>

Commit message: Add hazcams

File: models/lunar_pole_exploration_rover/urdf/chassis.xacro (robot description, xacro)
@@ -225,4 +225,96 @@
 		<origin xyz="-0.705 0.150 0.682" rpy="0 0 ${PI}"/>
 	</joint>
+	<link name="haz_camera_link_left_front">
+		<!-- Inertial for gazebo to take it into account, Put 1gr weight -->
+		<inertial>
+			<origin xyz="0 0 0" rpy="0 0 0"/>
+			<mass value="0.001" />
+			<inertia ixx="9.1875e-09" ixy="0.0" ixz="0.0" iyy="9.1875e-09" iyz="0.0" izz="1.378125e-08"/>
+		</inertial>
+		<visual>
+			<origin rpy="0.0 0 0" xyz="0 0 0"/>
+			<geometry>
+				<box size="0.0005 0.0005 0.0005"/>
+			</geometry>
+			<material name="camera_green"/>
+		</visual>
+	</link>
+	<gazebo reference="haz_camera_link_left_front">
+		<material>Gazebo/Green</material>
+	</gazebo>
+	<joint name="haz_camera_link_left_front_joint" type="fixed">
+		<parent link="body"/>
+		<child link="haz_camera_link_left_front"/>
+		<origin xyz="0.270 0.310 0.110" rpy="0 ${PI/4} ${PI/4}"/>
+	</joint>
+	<link name="haz_camera_link_left_rear">
+		<!-- Inertial for gazebo to take it into account, Put 1gr weight -->
+		<inertial>
+			<origin xyz="0 0 0" rpy="0 0 0"/>
+			<mass value="0.001" />
+			<inertia ixx="9.1875e-09" ixy="0.0" ixz="0.0" iyy="9.1875e-09" iyz="0.0" izz="1.378125e-08"/>
+		</inertial>
+		<visual>
+			<origin rpy="0.0 0 0" xyz="0 0 0"/>
+			<geometry>
+				<box size="0.0005 0.0005 0.0005"/>
+			</geometry>
+			<material name="camera_green"/>
+		</visual>
+	</link>
+	<gazebo reference="haz_camera_link_left_rear">
+		<material>Gazebo/Green</material>
+	</gazebo>
+	<joint name="haz_camera_link_left_rear_joint" type="fixed">
+		<parent link="body"/>
+		<child link="haz_camera_link_left_rear"/>
+		<origin xyz="-0.270 0.310 0.110" rpy="0 ${PI/4} ${PI/4 + PI/2}"/>
+	</joint>
+		<link name="haz_camera_link_right_front">
+		<!-- Inertial for gazebo to take it into account, Put 1gr weight -->
+		<inertial>
+			<origin xyz="0 0 0" rpy="0 0 0"/>
+			<mass value="0.001" />
+			<inertia ixx="9.1875e-09" ixy="0.0" ixz="0.0" iyy="9.1875e-09" iyz="0.0" izz="1.378125e-08"/>
+		</inertial>
+		<visual>
+			<origin rpy="0.0 0 0" xyz="0 0 0"/>
+			<geometry>
+				<box size="0.0005 0.0005 0.0005"/>
+			</geometry>
+			<material name="camera_green"/>
+		</visual>
+	</link>
+	<gazebo reference="haz_camera_link_right_front">
+		<material>Gazebo/Green</material>
+	</gazebo>
+	<joint name="haz_camera_link_right_front_joint" type="fixed">
+		<parent link="body"/>
+		<child link="haz_camera_link_right_front"/>
+		<origin xyz="0.270 -0.310 0.110" rpy="0 ${PI/4} ${-PI/4}"/>
+	</joint>
+		<link name="haz_camera_link_right_rear">
+		<!-- Inertial for gazebo to take it into account, Put 1gr weight -->
+		<inertial>
+			<origin xyz="0 0 0" rpy="0 0 0"/>
+			<mass value="0.001" />
+			<inertia ixx="9.1875e-09" ixy="0.0" ixz="0.0" iyy="9.1875e-09" iyz="0.0" izz="1.378125e-08"/>
+		</inertial>
+		<visual>
+			<origin rpy="0.0 0 0" xyz="0 0 0"/>
+			<geometry>
+				<box size="0.0005 0.0005 0.0005"/>
+			</geometry>
+			<material name="camera_green"/>
+		</visual>
+	</link>
+	<gazebo reference="haz_camera_link_right_rear">
+		<material>Gazebo/Green</material>
+	</gazebo>
+	<joint name="haz_camera_link_right_rear_joint" type="fixed">
+		<parent link="body"/>
+		<child link="haz_camera_link_right_rear"/>
+		<origin xyz="-0.270 -0.310 0.110" rpy="0 ${PI/4} ${-PI/4 - PI/2}"/>
+	</joint>
   </xacro:macro>
 </robot>
